File: pcb/flex-cap/flex-cap.kicad_pcb (KiCad board)
At the start: 2 copper layers, 82.4 x 20.1 mm, 9 parts, among them J1 Conn_01x06_Pin, U1 AD7147-1

Commit message: Make production files
Parts:
- moved J1 0.08 mm to (190.7, 102.9)
Changed lines of the file:
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@@
 		(tags "resistor")
 		(property "Reference" "R2"
-			(at -1.524 0 360)
+			(at -1.524 0 0)
 			(layer "F.SilkS")
 			(effects
@@
 		)
 		(property "Value" "2k2"
-			(at 0 1.17 360)
+			(at 0 1.17 0)
 			(layer "F.Fab")
 			(effects
@@
 		)
 		(fp_text user "${REFERENCE}"
-			(at 0 0 360)
+			(at 0 0 0)
 			(layer "F.Fab")
 			(effects
@@
 	(footprint "User_Footprints:FPC_6P_P0.5mm"
 		(layer "F.Cu")
-		(at 190.827 102.89)
+		(at 190.746 102.89)
 		(property "Reference" "J1"
-			(at 0 -1.31 0)
+			(at -5.453 1.25 0)
 			(unlocked yes)
 			(layer "F.SilkS")
@@
 		(sheetfile "flex-cap.kicad_sch")
 		(fp_line
-			(start -1.5 -0.5)
-			(end -1.5 3)
+			(start -4.9 -0.5)
+			(end -4.9 3)
 			(stroke
 				(width 0.1)
@@
 		)
 		(fp_line
-			(start -1.5 -0.5)
+			(start -4.9 -0.5)
 			(end 1.1 -0.5)
 			(stroke
@@
 		)
 		(fp_line
-			(start -1.5 3)
+			(start -4.9 3)
 			(end 1.1 3)
 			(stroke
@@
 			)
 		)
+		(fp_text user "Thickness: 0.2mm"
+			(at 1.278 2.647 0)
+			(unlocked yes)
+			(layer "User.1")
+			(effects
+				(font
+					(size 1 1)
+					(thickness 0.15)
+				)
+				(justify left bottom)
+			)
+		)
 		(fp_text user "Stiffener: Polymide"
 			(at 1.124 1.024 0)
@@
 			)
 		)
-		(fp_text user "Thickness: 0.2mm"
-			(at 1.524 2.524 0)
-			(unlocked yes)
-			(layer "User.1")
-			(effects
-				(font
-					(size 1 1)
-					(thickness 0.15)
-				)
-				(justify left bottom)
-			)
-		)
 		(pad "1" connect roundrect
-			(at 0 0)
-			(size 2 0.3)
+			(at -0.5 0)
+			(size 3.2 0.3)
 			(layers "B.Cu" "B.Mask")
 			(roundrect_rratio 0.25)
@@
 		)
 		(pad "2" connect roundrect
-			(at 0 0.499999)
-			(size 2 0.3)
+			(at -0.5 0.5)
+			(size 3.2 0.3)
 			(layers "B.Cu" "B.Mask")
 			(roundrect_rratio 0.25)
@@
 		)
 		(pad "3" connect roundrect
-			(at 0 1)
-			(size 2 0.3)
+			(at -0.5 1)
+			(size 3.2 0.3)
 			(layers "B.Cu" "B.Mask")
 			(roundrect_rratio 0.25)
@@
 		)
 		(pad "4" connect roundrect
-			(at 0 1.5)
-			(size 2 0.3)
+			(at -0.5 1.5)
+			(size 3.2 0.3)
 			(layers "B.Cu" "B.Mask")
 			(roundrect_rratio 0.25)
@@
 		)
 		(pad "5" connect roundrect
-			(at 0 2.000001)
-			(size 2 0.3)
+			(at -0.5 2)
+			(size 3.2 0.3)
 			(layers "B.Cu" "B.Mask")
 			(roundrect_rratio 0.25)
@@
 		)
 		(pad "6" connect roundrect
-			(at 0 2.5)
-			(size 2 0.3)
+			(at -0.5 2.5)
+			(size 3.2 0.3)
 			(layers "B.Cu" "B.Mask")
 			(roundrect_rratio 0.25)
@@
 		(tags "resistor")
 		(property "Reference" "R1"
-			(at -1.524 0 360)
+			(at -1.524 0 0)
 			(layer "F.SilkS")
 			(effects
@@
 		)
 		(property "Value" "2k2"
-			(at 0 1.17 360)
+			(at 0 1.17 0)
 			(layer "F.Fab")
 			(effects
@@
 		)
 		(fp_text user "${REFERENCE}"
-			(at 0 0 360)
+			(at 0 0 0)
 			(layer "F.Fab")
 			(effects
@@
 		(tags "resistor")
 		(property "Reference" "R3"
-			(at -1.524 0 360)
+			(at -1.524 0 0)
 			(layer "F.SilkS")
 			(effects
@@
 		)
 		(property "Value" "2k2"
-			(at 0 1.17 360)
+			(at 0 1.17 0)
 			(layer "F.Fab")
 			(effects
@@
 		)
 		(fp_text user "${REFERENCE}"
-			(at 0 0 360)
+			(at 0 0 0)
 			(layer "F.Fab")
 			(effects
@@
 					(thickness 0.15)
 				)
+			)
+		)
+		(property "LCSC" "C207411"
+			(at 0 0 45)
+			(unlocked yes)
+			(layer "F.Fab")
+			(hide yes)
+			(effects
+				(font
+					(size 1 1)
+					(thickness 0.15)
+				)
