File: pcb/flex-cap/flex-cap.kicad_sch (KiCad schematic)
At the start: 8 parts, among them U1 AD7147-1

Commit message: Finish schematic and pcb
Parts:
- added J1: Conn_01x06_Pin, User_Footprints:FPC_6P_P0.5mm, symbol Connector:Conn_01x06_Pin
- added TP0, TP1, TP10, TP11, TP12, TP13, TP2, TP3, TP4, TP5, TP6, TP7, TP8, TP9: TestPoint, symbol Connector:TestPoint
- U1: LCSC (none) -> C207411
Connections:
- net +3V3: now also J1.5 (Pin_5)
- net CIN0: now also TP0.1
- net CIN1: now also TP1.1
- net CIN10: now also TP10.1
- net CIN11: now also TP11.1
- net CIN12: now also TP12.1
- net CIN2: now also TP2.1
- net CIN3: now also TP3.1
- net CIN4: now also TP4.1
- net CIN5: now also TP5.1
- net CIN6: now also TP6.1
- net CIN7: now also TP7.1
- net CIN8: now also TP8.1
- net CIN9: now also TP9.1
- net GND: now also U1.25 (PAD), J1.1 (Pin_1), J1.6 (Pin_6)
- net INT: now also J1.2 (Pin_2)
- net SCL: now also J1.3 (Pin_3)
- net SDA: now also J1.4 (Pin_4)
- net SHLD: now also TP13.1
Other:
- moved on the sheet: C5, R1, R2, R3

Commit message: Fix pcb origins
Parts:
- J1: now not fitted; now left out of the parts list
Changed lines of the file:
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@@
 		(unit 1)
 		(exclude_from_sim no)
-		(in_bom yes)
+		(in_bom no)
 		(on_board yes)
-		(dnp no)
+		(dnp yes)
 		(property "Reference" "J1"
 			(at 146.05 63.5001 0)
